File: Intefaces/LocoNet/LocoNetInterface_V1.1/LocoNetInterface_V1.1.kicad_pcb (KiCad board)
At the start: 2 copper layers, 50 x 31 mm, 19 parts, among them J1 RJ12, J2 Conn_01x04, J3 RJ12, Q1 BC849, Q2 BC849, U1 LM311

Commit message: First Version
Routing:
- net +5V: track 0.00 -> 81.7 mm, vias 0 -> 3
- net Net-(J1-Pad1): track 0.00 -> 17.6 mm
- net Net-(J1-Pad6): track 0.00 -> 16.9 mm
- net GND: vias 0 -> 5
Changed lines of the file:
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@@
     (thickness 1.6)
     (drawings 6)
-    (tracks 71)
+    (tracks 110)
     (zones 0)
     (modules 19)
@@
       (rotate (xyz 0 0 0))
     )
+    (model ${KISYS3DMOD}/Connector_RJ.3dshapes/RJ12_Amphenol_54601.step
+      (offset (xyz 3.2 -16.75 0))
+      (scale (xyz 1 1 1))
+      (rotate (xyz -90 0 0))
+    )
   )
   (module Package_TO_SOT_SMD:SOT-23 (layer F.Cu)
@@
       (rotate (xyz 0 0 0))
     )
+    (model ${KISYS3DMOD}/Connector_RJ.3dshapes/RJ12_Amphenol_54601.step
+      (offset (xyz 3.2 -16.75 0))
+      (scale (xyz 1 1 1))
+      (rotate (xyz -90 0 0))
+    )
   )
   (module Resistor_SMD:R_1206_3216Metric (layer F.Cu)
@@
   (segment (start 81.15 124.32) (end 81.01 124.46) (width 0.25) (layer F.Cu) (net 4))
   (segment (start 85.1875 124.32) (end 81.15 124.32) (width 0.25) (layer F.Cu) (net 4))
+  (segment (start 55.46 111.35) (end 54.385 111.35) (width 0.25) (layer F.Cu) (net 5))
+  (segment (start 54.385 111.35) (end 53.975 111.76) (width 0.25) (layer F.Cu) (net 5))
+  (segment (start 53.975 124.865) (end 55.46 126.35) (width 0.25) (layer F.Cu) (net 5))
+  (segment (start 53.975 111.76) (end 53.975 124.865) (width 0.25) (layer F.Cu) (net 5))
+  (via (at 69.215 121.92) (size 0.8) (drill 0.4) (layers F.Cu B.Cu) (net 6))
+  (via (at 80.645 117.475) (size 0.8) (drill 0.4) (layers F.Cu B.Cu) (net 6))
+  (via (at 78.105 109.22) (size 0.8) (drill 0.4) (layers F.Cu B.Cu) (net 6))
+  (via (at 72.39 104.14) (size 0.8) (drill 0.4) (layers F.Cu B.Cu) (net 6))
+  (via (at 55.245 115.57) (size 0.8) (drill 0.4) (layers F.Cu B.Cu) (net 6))
   (segment (start 58.759999 121.780001) (end 61.099999 121.780001) (width 0.25) (layer F.Cu) (net 7))
   (segment (start 58 122.54) (end 58.759999 121.780001) (width 0.25) (layer F.Cu) (net 7))
@@
   (segment (start 56.545001 121.085001) (end 58 122.54) (width 0.25) (layer F.Cu) (net 7))
   (segment (start 56.545001 109.895001) (end 56.545001 121.085001) (width 0.25) (layer F.Cu) (net 7))
+  (segment (start 59.01 120) (end 59.69 119.32) (width 0.25) (layer B.Cu) (net 8))
+  (segment (start 58 120) (end 59.01 120) (width 0.25) (layer B.Cu) (net 8))
+  (segment (start 59.01 105) (end 58 105) (width 0.25) (layer B.Cu) (net 8))
+  (segment (start 59.69 105.68) (end 59.01 105) (width 0.25) (layer B.Cu) (net 8))
+  (segment (start 59.69 119.32) (end 59.69 105.68) (width 0.25) (layer B.Cu) (net 8))
+  (segment (start 85.895 111.76) (end 80.01 105.875) (width 0.25) (layer B.Cu) (net 9))
+  (segment (start 86.995 111.76) (end 85.895 111.76) (width 0.25) (layer B.Cu) (net 9))
+  (via (at 80.01 103.505) (size 0.8) (drill 0.4) (layers F.Cu B.Cu) (net 9))
+  (segment (start 80.01 105.875) (end 80.01 103.505) (width 0.25) (layer B.Cu) (net 9))
+  (segment (start 84.425 103.505) (end 84.6 103.68) (width 0.25) (layer F.Cu) (net 9))
+  (segment (start 80.01 103.505) (end 84.425 103.505) (width 0.25) (layer F.Cu) (net 9))
+  (segment (start 62.02571 103.14429) (end 61.33 103.84) (width 0.25) (layer F.Cu) (net 9))
+  (segment (start 62.53001 102.63999) (end 62.02571 103.14429) (width 0.25) (layer F.Cu) (net 9))
+  (segment (start 80.01 103.505) (end 79.14499 102.63999) (width 0.25) (layer F.Cu) (net 9))
+  (segment (start 80.01 105.875) (end 80.01 109.22) (width 0.25) (layer B.Cu) (net 9))
+  (via (at 66.04 111.125) (size 0.8) (drill 0.4) (layers F.Cu B.Cu) (net 9))
+  (segment (start 80.01 109.22) (end 78.105 111.125) (width 0.25) (layer B.Cu) (net 9))
+  (segment (start 78.105 111.125) (end 66.04 111.125) (width 0.25) (layer B.Cu) (net 9))
+  (segment (start 66.04 111.125) (end 66.04 112.9) (width 0.25) (layer F.Cu) (net 9))
+  (segment (start 85.895 111.76) (end 84.455 113.2) (width 0.25) (layer B.Cu) (net 9))
+  (segment (start 84.455 113.2) (end 84.455 128.27) (width 0.25) (layer B.Cu) (net 9))
+  (via (at 86.995 129.54) (size 0.8) (drill 0.4) (layers F.Cu B.Cu) (net 9))
+  (segment (start 84.455 128.27) (end 85.725 129.54) (width 0.25) (layer B.Cu) (net 9))
+  (segment (start 85.725 129.54) (end 86.995 129.54) (width 0.25) (layer B.Cu) (net 9))
+  (segment (start 87.4 129.135) (end 86.995 129.54) (width 0.25) (layer F.Cu) (net 9))
+  (segment (start 87.4 127.32) (end 87.4 129.135) (width 0.25) (layer F.Cu) (net 9))
+  (segment (start 79.14499 102.63999) (end 76.2 102.63999) (width 0.25) (layer F.Cu) (net 9))
+  (segment (start 76.2 102.63999) (end 62.53001 102.63999) (width 0.25) (layer F.Cu) (net 9))
+  (segment (start 75.09 103.74999) (end 76.2 102.63999) (width 0.25) (layer F.Cu) (net 9))
+  (segment (start 75.09 105.41) (end 75.09 103.74999) (width 0.25) (layer F.Cu) (net 9))
   (segment (start 73.79 127.635) (end 75.565 125.86) (width 0.25) (layer F.Cu) (net 10))
   (segment (start 62.865 125.86) (end 62.865 126.585) (width 0.25) (layer F.Cu) (net 10))

Commit message: Loconet JLPCB
Parts:
- D1, D2: footprint LED_SMD:LED_0603_1608Metric_Castellated -> LED_SMD:LED_0805_2012Metric
- J1, J3: footprint Connector_RJ:RJ12_Amphenol_54601 -> LocoNetInterface_V1:AMPHENOL_RJE0166001
- J2: footprint Connector_PinHeader_2.54mm:PinHeader_1x04_P2.54mm_Vertical -> Connector_JST:JST_XH_B4B-XH-A_1x04_P2.50mm_Vertical
- Q1, Q2: value BC849 -> 2N3904
- R1, R10, R11, R2, R3, R4, R5, R6, R7, R8, R9: footprint Resistor_SMD:R_1206_3216Metric -> Resistor_SMD:R_0805_2012Metric
- moved J3 10.1 mm to (48.5, 123.5)
- moved J1 9.76 mm to (48.5, 107.2)
- moved J2 7.56 mm to (86.0, 119.2), turned to 90 degrees
- turned R8 to 180 degrees
Connections:
- J2 pad 2: /RX -> /TX
- J2 pad 3: /TX -> /RX
Routing:
- net Net-(J1-Pad6): track 16.9 -> 26.2 mm
- net +5V: track 81.7 -> 76.6 mm
- net /loconet: track 47.8 -> 51.5 mm
- net Net-(J1-Pad1): track 17.6 -> 20.1 mm
- net Net-(R4-Pad2): track 15.9 -> 16.9 mm
- net Net-(D2-Pad2): track 4.02 -> 3.13 mm
- net GND: vias 5 -> 7
Other:
- board text added: "Gnd Rx Tx 5V"
- board text removed: "5V Rx Tx Gnd"
