File: dcc-turnout/board/DccDecoderIt2/DccDecoder.kicad_pcb (KiCad board)
At the start: 4 copper layers, 95 x 30 mm, 67 parts, among them J1 Conn_01x02, J10 Conn_01x01, J11 Conn_01x02, J12 Conn_01x01, J13 Conn_01x01, J14 Conn_01x02, J15 Conn_01x03, J16 Conn_01x02, J17 Conn_01x04, J2 Conn_01x02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

Commit message: Fab iteration
Parts:
- C1, C2, C3, C4, C5, C6, C7, C8, C9: footprint Capacitor_SMD:C_1206_3216Metric -> Capacitor_SMD:C_0805_2012Metric
- D1, D2, D3, D4: footprint LED_SMD:LED_1206_3216Metric -> LED_SMD:LED_0805_2012Metric
- L1: footprint Inductor_SMD:L_1206_3216Metric -> Inductor_SMD:L_0805_2012Metric
- Q1, Q2, Q4, Q6: value NXV55UNR -> AO3400A
- Q3, Q5: value NXV90EPR -> AO3401A
- R1: value 900 -> 1K; footprint Resistor_SMD:R_1206_3216Metric -> Resistor_SMD:R_0805_2012Metric
- R10, R11, R12, R13, R14, R15, R16, R17, R18, R2, R3, R4, R5, R6, R7, R8, R9: footprint Resistor_SMD:R_1206_3216Metric -> Resistor_SMD:R_0805_2012Metric
- moved R6 8.54 mm to (101.0, 55.0)
- moved R7 5.83 mm to (101.0, 57.0), turned to 0 degrees
- moved R2 3.59 mm to (61.0, 49.9)
- moved R3 3.59 mm to (65.0, 49.9)
- moved R1 3.50 mm to (57.0, 50.0)
- moved R16 2.09 mm to (77.5, 46.4)
- moved R5 1.96 mm to (101.0, 61.5)
- moved R8 1.80 mm to (47.5, 53.0)
- moved C4 1.62 mm to (98.0, 59.5)
- moved C7 1.50 mm to (96.0, 59.5)
- moved R11 1.04 mm to (47.6, 58.5)
- moved R9 1.01 mm to (36.1, 51.0)
- moved C2 1.00 mm to (94.0, 49.7)
- moved D1 1.00 mm to (57.0, 46.5)
- moved D2 1.00 mm to (61.0, 46.5)
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Routing:
- net /CfgStatus: track 13.6 -> 20.5 mm
- net /SDA: track 35.1 -> 39.7 mm
- net +3V3: track 71.8 -> 67.3 mm
- net /SCL: track 29.6 -> 26.3 mm
- net /ThrownLed: track 40.1 -> 43.3 mm
- net Net-(Q1-Pad1): track 4.17 -> 2.50 mm
- net /ClosedLed: track 46.2 -> 47.9 mm
- net Net-(D3-Pad1): track 3.14 -> 1.56 mm
- net Net-(D2-Pad1): track 3.14 -> 1.56 mm
- net Net-(D1-Pad1): track 3.14 -> 1.65 mm
- net /uC 030K6/NRST: track 72.3 -> 71.0 mm
- net /uC 030K6/_VDDA: track 15.5 -> 14.5 mm
- net /ReleEn: track 46.6 -> 47.5 mm
- net /uC 030K6/PF0: track 10.8 -> 9.85 mm
- net /uC 030K6/PF1: track 11.6 -> 10.7 mm
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Other:
- board text added: "CLK"
