File: DccBlocks/IndicartorLeds/Study/Study.kicad_pcb (KiCad board)
At the start: 2 copper layers, 10 x 23.5 mm, 4 parts

Commit message: "Udpated to reduce size"
Parts:
- added REF**: PinHeader_1x03_P2.00mm_Vertical, Connector_PinHeader_2.00mm:PinHeader_1x03_P2.00mm_Vertical, F.Cu at (48.0, 53.6)
- added REF**: LED_WS2812B_PLCC4_5.0x5.0mm_P3.2mm, LED_SMD:LED_WS2812B_PLCC4_5.0x5.0mm_P3.2mm, F.Cu at (111.0, 29.0)
- added REF**: PinHeader_1x03_P2.54mm_Vertical, Connector_PinHeader_2.54mm:PinHeader_1x03_P2.54mm_Vertical, F.Cu at (109.5, 85.6)
- added REF**: PinHeader_1x03_P2.54mm_Vertical, Connector_PinHeader_2.54mm:PinHeader_1x03_P2.54mm_Vertical, F.Cu at (109.5, 64.4)
- added REF**: LED_WS2812B_PLCC4_5.0x5.0mm_P3.2mm, LED_SMD:LED_WS2812B_PLCC4_5.0x5.0mm_P3.2mm, F.Cu at (112.0, 81.0)
- added REF**: LED_WS2812B_PLCC4_5.0x5.0mm_P3.2mm, LED_SMD:LED_WS2812B_PLCC4_5.0x5.0mm_P3.2mm, F.Cu at (112.0, 69.0)
- added REF**: LED_WS2812B_PLCC4_5.0x5.0mm_P3.2mm, LED_SMD:LED_WS2812B_PLCC4_5.0x5.0mm_P3.2mm, F.Cu at (112.0, 75.0)
- added REF**: LED_WS2812B_PLCC4_5.0x5.0mm_P3.2mm, LED_SMD:LED_WS2812B_PLCC4_5.0x5.0mm_P3.2mm, F.Cu at (111.0, 35.0)
- added REF**: PinHeader_2x03_P2.54mm_Vertical, Connector_PinHeader_2.54mm:PinHeader_2x03_P2.54mm_Vertical, F.Cu at (108.5, 48.2)
- added REF**: LED_WS2812B_PLCC4_5.0x5.0mm_P3.2mm, LED_SMD:LED_WS2812B_PLCC4_5.0x5.0mm_P3.2mm, F.Cu at (111.0, 41.0)
Routing:
- net (no net): track 89.6 -> 269.6 mm, vias 6 -> 18
Other:
- board size 10 x 23.5 mm -> 72 x 63.5 mm
- board text added: "Grid 6 m"
