File: dcc-turnout/board/DccDecoder0805/DccDecoder.kicad_sch (KiCad schematic)
At the start: 22 parts, among them J1 Conn_01x02, J2 Conn_01x02, J3 Conn_01x02, J4 Conn_01x04, J7 Conn_01x06, J8 Conn_01x03

Commit message: Updates y mejoras
Other:
- title: (none) -> DCC Decoder Turnout
Changed lines of the file:
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@@
 (kicad_sch (version 20211123) (generator eeschema)
   (paper "A4")
+  (title_block
+    (title "DCC Decoder Turnout")
+    (date "2022-07-04")
+    (rev "0.4.1")
+  )
   (junction (at 274.32 135.89) (diameter 0) (color 0 0 0 0)
   )
