File: dcc-turnout/board/DccDecoder0805/OutPuts.kicad_sch (KiCad schematic)
At the start: 28 parts, among them J10 Conn_01x01, J11 Conn_01x02, J12 Conn_01x01, J13 Conn_01x01, J14 Conn_01x02, J15 Conn_01x03, J16 Conn_01x02, J17 Conn_01x04, J9 Conn_01x01, Q1 AO3400A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

Commit message: Updates y mejoras
Other:
- title: (none) -> DCC Decoder Turnout
Changed lines of the file:
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@@
 (kicad_sch (version 20211123) (generator eeschema)
   (paper "A4")
+  (title_block
+    (title "DCC Decoder Turnout")
+    (date "2022-07-04")
+    (rev "0.4.1")
+  )
   (junction (at 148.59 59.69) (diameter 0) (color 0 0 0 0)
   )
