File: dcc-turnout/board/DccDecoder0805/STM32F030K6.kicad_sch (KiCad schematic)
At the start: 16 parts, among them J6 Conn_02x05 Odd_Even, SW1 SW_Push, U1 STM32F030K6Tx, Y1 8MHz

Commit message: Updates y mejoras
Other:
- title: (none) -> DCC Decoder Turnout
Changed lines of the file:
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@@
 (kicad_sch (version 20211123) (generator eeschema)
   (paper "A4")
+  (title_block
+    (title "DCC Decoder Turnout")
+    (date "2022-07-04")
+    (rev "0.4.1")
+  )
   (junction (at 208.28 85.09) (diameter 0) (color 0 0 0 0)
   )
