File: DccBlocks/DccPowerDistribution/board/PowerDist.kicad_sch (KiCad schematic)
At the start: 33 parts, among them J3 Conn_01x03, Q2 BC817, Q3 2N7002, Q4 BSS308, U1 AMS1117-3.3, U4 TPS54331D

Commit message: Update kibot, clean drc,...
Parts:
- C1, C14, C15, C16, C2, C4: symbol Device:CP -> Device:C_Polarized
Changed lines of the file:
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@@
     (pin "3")
   )
-  (symbol (lib_id "Device:CP") (at 157.48 38.1 0) (unit 1)
+  (symbol (lib_id "Device:C_Polarized") (at 157.48 38.1 0) (unit 1)
     (in_bom yes) (on_board yes)
     (property "Reference" "C4" (id 0) (at 160.4772 36.9316 0)
@@
     (pin "2")
   )
-  (symbol (lib_id "Device:CP") (at 125.73 38.1 0) (unit 1)
+  (symbol (lib_id "Device:C_Polarized") (at 125.73 38.1 0) (unit 1)
     (in_bom yes) (on_board yes)
     (property "Reference" "C2" (id 0) (at 128.7272 36.9316 0)
@@
     (pin "2")
   )
-  (symbol (lib_id "Device:CP") (at 201.93 27.94 0) (unit 1)
+  (symbol (lib_id "Device:C_Polarized") (at 201.93 27.94 0) (unit 1)
     (in_bom yes) (on_board yes)
     (property "Reference" "C1" (id 0) (at 204.9272 26.7716 0)
@@
     (pin "1")
   )
-  (symbol (lib_id "Device:CP") (at 223.52 27.94 0) (unit 1)
+  (symbol (lib_id "Device:C_Polarized") (at 223.52 27.94 0) (unit 1)
     (in_bom yes) (on_board yes)
     (property "Reference" "C15" (id 0) (at 226.5172 26.7716 0)
@@
     (pin "2")
   )
-  (symbol (lib_id "Device:CP") (at 212.09 27.94 0) (unit 1)
+  (symbol (lib_id "Device:C_Polarized") (at 212.09 27.94 0) (unit 1)
     (in_bom yes) (on_board yes)
     (property "Reference" "C14" (id 0) (at 215.0872 26.7716 0)
@@
     (pin "2")
   )
-  (symbol (lib_id "Device:CP") (at 273.05 31.75 0) (unit 1)
+  (symbol (lib_id "Device:C_Polarized") (at 273.05 31.75 0) (unit 1)
     (in_bom yes) (on_board yes)
     (property "Reference" "C16" (id 0) (at 276.0472 30.5816 0)

Commit message: Updates
Changed lines of the file:
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@@
     (effects (font (size 1.27 1.27)) (justify left bottom))
   )
-  (label "_DccVin" (at 25.4 57.15 180)
+  (label "DccVin" (at 25.4 57.15 180)
     (effects (font (size 1.27 1.27)) (justify right bottom))
   )
-  (label "_Vdrive" (at 25.4 54.61 180)
+  (label "Vdrive" (at 25.4 54.61 180)
     (effects (font (size 1.27 1.27)) (justify right bottom))
   )
-  (label "_3V" (at 57.15 31.75 180)
+  (label "3.3V" (at 57.15 31.75 180)
     (effects (font (size 1.27 1.27)) (justify right bottom))
   )
-  (label "_5V" (at 109.22 29.21 180)
+  (label "5V" (at 109.22 29.21 180)
     (effects (font (size 1.27 1.27)) (justify right bottom))
   )
-  (label "_Vdrive" (at 275.59 22.86 0)
+  (label "Vdrive" (at 275.59 22.86 0)
     (effects (font (size 1.27 1.27)) (justify left bottom))
   )
@@
     (effects (font (size 1.27 1.27)) (justify left bottom))
   )
-  (label "_5V" (at 215.9 81.28 180)
+  (label "5V" (at 215.9 81.28 180)
     (effects (font (size 1.27 1.27)) (justify right bottom))
   )
-  (label "_3V" (at 172.72 27.94 180)
+  (label "3.3V" (at 172.72 27.94 180)
     (effects (font (size 1.27 1.27)) (justify right bottom))
   )
-  (label "_DccVin" (at 33.02 30.48 0)
+  (label "DccVin" (at 33.02 30.48 0)
     (effects (font (size 1.27 1.27)) (justify left bottom))
   )
@@
     (effects (font (size 1.27 1.27)) (justify left bottom))
   )
-  (label "_Vin" (at 33.02 24.13 0)
+  (label "Vin" (at 33.02 24.13 0)
     (effects (font (size 1.27 1.27)) (justify left bottom))
   )
-  (label "_Vin" (at 66.04 57.15 180)
+  (label "Vin" (at 66.04 57.15 180)
     (effects (font (size 1.27 1.27)) (justify right bottom))
   )
-  (label "_Vdrive" (at 80.01 57.15 0)
+  (label "Vdrive" (at 80.01 57.15 0)
     (effects (font (size 1.27 1.27)) (justify left bottom))
   )
-  (label "_DccVin" (at 190.5 22.86 180)
+  (label "DccVin" (at 190.5 22.86 180)
     (effects (font (size 1.27 1.27)) (justify right bottom))
   )
-  (label "_Vdrive" (at 57.15 24.13 180)
+  (label "Vdrive" (at 57.15 24.13 180)
     (effects (font (size 1.27 1.27)) (justify right bottom))
   )
-  (label "_Vin" (at 191.77 48.26 180)
+  (label "Vin" (at 191.77 48.26 180)
     (effects (font (size 1.27 1.27)) (justify right bottom))
   )
-  (label "_5V" (at 57.15 27.94 180)
+  (label "5V" (at 57.15 27.94 180)
     (effects (font (size 1.27 1.27)) (justify right bottom))
   )
-  (label "_Vin" (at 25.4 52.07 180)
+  (label "Vin" (at 25.4 52.07 180)
     (effects (font (size 1.27 1.27)) (justify right bottom))
   )
@@
     (effects (font (size 1.27 1.27)) (justify left bottom))
   )
-  (label "_Vdrive" (at 49.53 77.47 180)
+  (label "Vdrive" (at 49.53 77.47 180)
     (effects (font (size 1.27 1.27)) (justify right bottom))
   )

Commit message: Update Kibot Scripts to latest versions
Parts:
- C1, C2, C4: LCSC C7171 -> (none); LCSC# (none) -> C7171; MNF# (none) -> T494A106M020AT; Mouser 80-T494A106M020 -> (none); Mouser# (none) -> 80-T494A106M020; REF T494A106M020AT -> (none)
- C10: value 100nf 1m -> 100nf; Farnell 2581103 -> (none); Farnell# (none) -> 2581103; MNF# (none) -> C1206C104M5RACTU; REF C1206C104M5RACTU -> (none); Tolerance (none) -> 1mO
- C11, C12, C13, C5, C7: value 10uf 2m -> 10uf; MNF# (none) -> CL31A106KPHNNNE; Mouser 187-CL31A106KPHNNNE -> (none); Mouser# (none) -> 187-CL31A106KPHNNNE; REF CL31A106KPHNNNE -> (none); Tolerance (none) -> 2mO
- C14, C15, C16: MNF# (none) -> 865060445005; REF 865060445005 -> (none)
- C6: Farnell 2497123 -> (none); Farnell# (none) -> 2497123; MNF# (none) -> 1206N100J500CT; REF 1206N100J500CT -> (none)
- C8: Farnell 1759347 -> (none); Farnell# (none) -> 1759347; MNF# (none) -> MC1206B562K500CT; REF MC1206B562K500CT -> (none)
- C9: Farnell 1759349 -> (none); Farnell# (none) -> 1759349; MNF# (none) -> MC1206B822K500CT; REF MC1206B822K500CT -> (none)
- D2, D3, D8: MNF# (none) -> GS1510FL_R1_00001; Mouser 241-GS1510FLR100001 -> (none); Mouser# (none) -> 241-GS1510FLR100001; REF GS1510FL_R1_00001 -> (none)
- D7: Farnell 2748189 -> (none); Farnell# (none) -> 2748189; MNF# (none) -> SS24A+; REF SS24A+ -> (none)
- J3: value Conn_01x03 -> Pin_01x03; Farnell# (none) -> 1098611; MNF# (none) -> 1776275-2
- L1: value 22uH 75mO -> 22uH; Farnell 2434023 -> (none); Farnell# (none) -> 2434023; MNF# (none) -> SRP1038A-220M; REF SRP1038A-220M -> (none); Tolerance (none) -> 75mO
- Q2: MNF# (none) -> BC817-25,215; Mouser 771-BC817-25-T/R -> (none); Mouser# (none) -> 771-BC817-25-T/R; REF BC817-25,215 -> (none)
- Q4: MNF# (none) -> BSS308PE H6327; Mouser 726-BSS308PEH6327 -> (none); Mouser# (none) -> 726-BSS308PEH6327; REF BSS308PE H6327 -> (none)
- R11: Farnell 2695169 -> (none); Farnell# (none) -> 2695169; MNF# (none) -> ERJ8ENF5621V; REF ERJ8ENF5621V -> (none)
- R12: Farnell 2307301 -> (none); Farnell# (none) -> 2307301; MNF# (none) -> ERJ8ENF1022V; REF ERJ8ENF1022V -> (none)
- R13: Farnell 2307494 -> (none); Farnell# (none) -> 2307494; MNF# (none) -> ERJ8ENF1961V; REF ERJ8ENF1961V -> (none)
- U1: LCSC C6186 -> (none); LCSC# (none) -> C6186; MNF# (none) -> NCP1117LPST33T3G; Mouser 863-NCP1117LPST33T3G -> (none); Mouser# (none) -> 863-NCP1117LPST33T3G; REF NCP1117LPST33T3G -> (none)
- U4: Farnell 1645383 -> (none); Farnell# (none) -> 1645383; MNF# (none) -> TPS54331D; REF TPS54331D -> (none)
