File: MimicPanel/Stm32F103Board/Stm32F103Board.kicad_pcb (KiCad board)
At the start: 2 copper layers, 104 x 77 mm, 30 parts, among them J1 Conn_01x03, J10 Conn_01x06, J11 Conn_01x04, J12 Conn_01x06, J13 Conn_01x06, J14 Conn_01x03, J15 Conn_01x08, J16 Conn_01x08, J17 Conn_02x08_Odd_Even, J18 Conn_02x08_Odd_Even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

Commit message: mimic Panel Update
Other:
- net class Default removed
- net class Power removed
