File: DccBlocks/ABC/AbcStop/AbcStop.kicad_pcb (KiCad board)
At the start: 2 copper layers, 51 x 18 mm, 8 parts, among them J1 SCREW, J2 43650-0200

Commit message: AbcStop
Parts:
- added C1: 4.7uF, Capacitor_SMD:CP_Elec_4x5.4, F.Cu at (66.0, 45.2)
- added D6: 1N4148, Diode_SMD:D_SOD-323, F.Cu at (93.5, 52.5)
- added D8: ES1G+, Diode_SMD:D_SMA, F.Cu at (63.0, 53.5)
- added J3: Conn_01x02, Connector_PinHeader_2.54mm:PinHeader_1x02_P2.54mm_Vertical, F.Cu at (85.0, 56.8)
- added J4: Conn_01x02, Connector_PinHeader_2.54mm:PinHeader_1x02_P2.54mm_Vertical, F.Cu at (78.5, 37.5)
- added Q1: PSMN022, DigitalTrains:sot404, F.Cu at (75.5, 50.5)
- added Q2: Q_PMOS_GSD, Package_TO_SOT_SMD:SOT-23, F.Cu at (96.7, 56.8)
- added Q3: PSMN022, DigitalTrains:sot404, F.Cu at (106.7, 50.5)
- added R1: 1K, Resistor_SMD:R_1206_3216Metric_Pad1.30x1.75mm_HandSolder, F.Cu at (94.5, 45.0)
- added R2: 3K, Resistor_SMD:R_1206_3216Metric_Pad1.30x1.75mm_HandSolder, F.Cu at (96.7, 60.5)
- added R3: 1K, Resistor_SMD:R_1206_3216Metric_Pad1.30x1.75mm_HandSolder, F.Cu at (92.0, 59.0)
- added R4: 3K, Resistor_SMD:R_1206_3216Metric_Pad1.30x1.75mm_HandSolder, F.Cu at (86.0, 38.2)
- added TP1: TestPoint, TestPoint:TestPoint_Pad_D1.5mm, F.Cu at (114.2, 45.2)
- added U1: VO615A, Package_DIP:SMDIP-4_W9.53mm, F.Cu at (86.2, 48.5)
- J2: value 43650-0200 -> SCREW; footprint DigitalTrains:MOLEX_436500200 -> TerminalBlock_Phoenix:TerminalBlock_Phoenix_PT-1,5-2-3.5-H_1x02_P3.50mm_Horizontal
- NT1: moved to B.Cu
- moved J2 16.1 mm to (120.0, 60.0), turned to -90 degrees
- moved D1 6.25 mm to (100.2, 68.0)
- moved D2 6.25 mm to (93.2, 70.0)
- moved D3 6.25 mm to (83.2, 70.0)
- moved D4 6.25 mm to (76.2, 68.0)
- moved D5 6.25 mm to (88.2, 66.0)
- moved NT1 4.25 mm to (86.2, 60.0)
Routing:
- net /High_Right: track 0.00 -> 60.4 mm, vias 0 -> 2
- net /Right_IN: track 18.0 -> 74.6 mm
- net Net-(D6-K): track 0.00 -> 49.2 mm
- net /Right_1: track 0.00 -> 42.4 mm
- net /Right_OUT: track 17.2 -> 49.6 mm
- net /Left_OUT: track 16.0 -> 31.7 mm
- net /enGnd: track 0.00 -> 10.5 mm, vias 0 -> 1
- net Net-(R4-Pad1): track 0.00 -> 9.44 mm, vias 0 -> 2
- net /Left_IN: track 17.0 -> 25.5 mm
- net Net-(J3-Pin_2): track 0.00 -> 8.21 mm
- net /GRight: track 0.00 -> 6.28 mm
- net Net-(D6-A): track 0.00 -> 5.25 mm
- net /en: track 0.00 -> 3.75 mm
Other:
- board size 51 x 18 mm -> 65.8 x 37.8 mm

Commit message: AbcStop Cleanup And Minor code change
Parts:
- moved J2 3.77 mm to (118.5, 63.5), turned to 90 degrees
Connections:
- J2 pad 1: /Left_OUT -> /Right_OUT
- J2 pad 2: /Right_OUT -> /Left_OUT
Routing:
- net /Right_OUT: track 49.6 -> 46.8 mm
- net /Left_OUT: track 31.7 -> 30.3 mm
Changed lines of the file:
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@@
     (property "ki_keywords" "R res resistor")
     (attr smd)
-    (fp_text reference "R2" (at 0 -1.82) (layer "F.SilkS")
+    (fp_text reference "R2" (at 0 2) (layer "F.SilkS")
         (effects (font (size 1 1) (thickness 0.15)))
     )
@@
     (property "ki_keywords" "diode")
     (attr smd)
-    (fp_text reference "D4" (at 3 3 -180) (layer "F.SilkS")
+    (fp_text reference "D4" (at -0.75 2.5 -90) (layer "F.SilkS")
         (effects (font (size 1 1) (thickness 0.15)))
     )
@@
     (property "ki_keywords" "connector")
     (attr through_hole)
-    (fp_text reference "J3" (at 0 -2.33 90) (layer "F.SilkS")
+    (fp_text reference "J3" (at -2.5 1.275 180) (layer "F.SilkS")
         (effects (font (size 1 1) (thickness 0.15)))
     )
@@
     (property "ki_keywords" "diode")
     (attr smd)
-    (fp_text reference "D3" (at 0 -2.5) (layer "F.SilkS")
+    (fp_text reference "D3" (at -4.25 0 90) (layer "F.SilkS")
         (effects (font (size 1 1) (thickness 0.15)))
     )
@@
     (property "ki_keywords" "R res resistor")
     (attr smd)
-    (fp_text reference "R3" (at 0 -1.82 90) (layer "F.SilkS")
+    (fp_text reference "R3" (at -3.5 0.05) (layer "F.SilkS")
         (effects (font (size 1 1) (thickness 0.15)))
     )
@@
     (property "ki_keywords" "diode")
     (attr smd)
-    (fp_text reference "D5" (at 0 3) (layer "F.SilkS")
+    (fp_text reference "D5" (at -4.5 1.5) (layer "F.SilkS")
         (effects (font (size 1 1) (thickness 0.15)))
     )
@@
   )
   (footprint "TerminalBlock_Phoenix:TerminalBlock_Phoenix_PT-1,5-2-3.5-H_1x02_P3.50mm_Horizontal" (layer "F.Cu")
-    (at 119.9501 60 -90)
+    (at 118.55 63.5 90)
     (descr "Terminal Block Phoenix PT-1,5-2-3.5-H, 2 pins, pitch 3.5mm, size 7x7.6mm^2, drill diamater 1.2mm, pad diameter 2.4mm, see , script-generated using https://github.com/pointhi/kicad-footprint-generator/scripts/TerminalBlock_Phoenix")
     (tags "THT Terminal Block Phoenix PT-1,5-2-3.5-H pitch 3.5mm size 7x7.6mm^2 drill 1.2mm pad 2.4mm")
@@
     (fp_circle (center 3.5 0) (end 5 0)
       (stroke (width 0.1) (type solid)) (fill none) (layer "F.Fab"))
-    (pad "1" thru_hole rect (at 0 0 270) (size 2.4 2.4) (drill 1.2) (layers "*.Cu" "*.Mask")
-      (net 7 "/Left_OUT") (pinfunction "Pin_1") (pintype "passive"))
-    (pad "2" thru_hole circle (at 3.5 0 270) (size 2.4 2.4) (drill 1.2) (layers "*.Cu" "*.Mask")
-      (net 2 "/Right_OUT") (pinfunction "Pin_2") (pintype "passive"))
+    (pad "1" thru_hole rect (at 0 0 90) (size 2.4 2.4) (drill 1.2) (layers "*.Cu" "*.Mask")
+      (net 2 "/Right_OUT") (pinfunction "Pin_1") (pintype "passive"))
+    (pad "2" thru_hole circle (at 3.5 0 90) (size 2.4 2.4) (drill 1.2) (layers "*.Cu" "*.Mask")
+      (net 7 "/Left_OUT") (pinfunction "Pin_2") (pintype "passive"))
     (model "${KICAD6_3DMODEL_DIR}/TerminalBlock_Phoenix.3dshapes/TerminalBlock_Phoenix_PT-1,5-2-3.5-H_1x02_P3.50mm_Horizontal.wrl"
       (offset (xyz 0 0 0))
@@
     (property "ki_keywords" "diode")
     (attr smd)
-    (fp_text reference "D1" (at -3 3 180) (layer "F.SilkS")
+    (fp_text reference "D1" (at -0.25 2.75 270) (layer "F.SilkS")
         (effects (font (size 1 1) (thickness 0.15)))
     )
@@
     (property "ki_keywords" "diode")
     (attr smd)
-    (fp_text reference "D2" (at 0 -2.5) (layer "F.SilkS")
+    (fp_text reference "D2" (at -4.25 0 90) (layer "F.SilkS")
         (effects (font (size 1 1) (thickness 0.15)))
     )
@@
   (gr_rect (start 58 35.25) (end 123.75 73)
     (stroke (width 0.1) (type default)) (fill none) (layer "Edge.Cuts"))
-  (gr_text "AbcStop 0.0.1\nJLCJLCJLCJLC" (at 73 60) (layer "F.SilkS")
+  (gr_text "AbcStop 0.0.1\nJLCJLCJLCJLC" (at 111 39) (layer "F.SilkS")
     (effects (font (size 1 1) (thickness 0.15)) (justify left bottom))
   )
@@
   (segment (start 112.75 63.5) (end 110.25 66) (width 1.5) (layer "F.Cu") (net 2))
   (segment (start 90.25 66) (end 100.25 66) (width 1.5) (layer "F.Cu") (net 2))
+  (segment (start 117.4501 63.5) (end 118.55 63.5) (width 1.5) (layer "F.Cu") (net 2))
   (segment (start 106.7001 56.0499) (end 114.25 56.0499) (width 1.5) (layer "F.Cu") (net 2))
-  (segment (start 117.4501 63.5) (end 119.9501 63.5) (width 1.5) (layer "F.Cu") (net 2))
   (segment (start 114.25 56.0499) (end 115.7001 57.5) (width 1.5) (layer "F.Cu") (net 2))
+  (segment (start 118.55 63.5) (end 112.75 63.5) (width 1.5) (layer "F.Cu") (net 2))
   (segment (start 115.7001 61.75) (end 117.4501 63.5) (width 1.5) (layer "F.Cu") (net 2))
-  (segment (start 119.9501 63.5) (end 112.75 63.5) (width 1.5) (layer "F.Cu") (net 2))
   (segment (start 110.25 66) (end 100.25 66) (width 1.5) (layer "F.Cu") (net 2))
   (segment (start 85.25 70) (end 91.25 70) (width 1.5) (layer "F.Cu") (net 3))
@@
   (segment (start 63 60) (end 63 55.75) (width 1.5) (layer "F.Cu") (net 6))
   (segment (start 84.25 60) (end 63 60) (width 1.5) (layer "B.Cu") (net 6))
-  (segment (start 88.25 60) (end 119.9501 60) (width 1.5) (layer "B.Cu") (net 7))
+  (segment (start 118.55 60) (end 88.25 60) (width 1.5) (layer "B.Cu") (net 7))
   (segment (start 66 43.45) (end 64.3 43.45) (width 0.5) (layer "F.Cu") (net 8))
   (segment (start 69.7 43.45) (end 69.75 43.5) (width 0.5) (layer "F.Cu") (net 8))

Commit message: AbcStop 0.0.2
Other:
- board text added: "AbcStop 0.0.2 JLCJLCJLCJLC"
- board text removed: "AbcStop 0.0.1 JLCJLCJLCJLC"
Changed lines of the file:
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@@
     (title "AbcStop")
     (date "2023-06-01")
-    (rev "0.0.1")
+    (rev "0.0.2")
     (company "Dcc Diy Tools")
   )
@@
   (gr_rect (start 58 35.25) (end 123.75 73)
     (stroke (width 0.1) (type default)) (fill none) (layer "Edge.Cuts"))
-  (gr_text "AbcStop 0.0.1\nJLCJLCJLCJLC" (at 111 39) (layer "F.SilkS")
+  (gr_text "AbcStop 0.0.2\nJLCJLCJLCJLC" (at 111 39) (layer "F.SilkS")
     (effects (font (size 1 1) (thickness 0.15)) (justify left bottom))
   )
