File: DccBlocks/ABC/AbcStop/AbcStop.kicad_sch (KiCad schematic)
At the start: 8 parts, among them J1 SCREW, J2 43650-0200

Commit message: AbcStop
Parts:
- added C1: 4.7uF, Capacitor_SMD:CP_Elec_4x5.4, symbol Device:C_Polarized
- added D6: 1N4148, Diode_SMD:D_SOD-323, symbol Diode:1N4148
- added D8: ES1G+, Diode_SMD:D_SMA, symbol Device:D
- added J3, J4: Conn_01x02, Connector_PinHeader_2.54mm:PinHeader_1x02_P2.54mm_Vertical, symbol Connector_Generic:Conn_01x02
- added Q1, Q3: PSMN022, DigitalTrains:sot404, symbol Device:Q_NMOS_GDS
- added Q2: Q_PMOS_GSD, Package_TO_SOT_SMD:SOT-23, symbol Device:Q_PMOS_GSD
- added R1, R3: 1K, Resistor_SMD:R_1206_3216Metric_Pad1.30x1.75mm_HandSolder, symbol Device:R
- added R2, R4: 3K, Resistor_SMD:R_1206_3216Metric_Pad1.30x1.75mm_HandSolder, symbol Device:R
- added TP1: TestPoint, TestPoint:TestPoint_Pad_D1.5mm, symbol Connector:TestPoint
- added U1: VO615A, Package_DIP:SMDIP-4_W9.53mm, symbol Isolator:VO615A
- J2: value 43650-0200 -> SCREW; footprint DigitalTrains:MOLEX_436500200 -> TerminalBlock_Phoenix:TerminalBlock_Phoenix_PT-1,5-2-3.5-H_1x02_P3.50mm_Horizontal
Connections:
- net Left_IN: now also D8.2 (A)
- net Right_IN: now also C1.2, J3.1 (Pin_1), Q1.2 (D), U1.3
- net Right_OUT: now also Q3.2 (D)
- new net: R4.1, U1.1
- new net: D6.2 (A), Q2.3 (D)
- new net: J3.2 (Pin_2), R3.2, U1.4
- new net: D6.1 (K), Q1.1 (G), Q3.1 (G), R1.1, TP1.1
- new net GRight: Q2.1 (G), R2.1, R3.1
- new net High_Right: C1.1, D8.1 (K), Q2.2 (S), R2.2
- new net Right_1: Q1.3 (S), Q3.3 (S), R1.2
- new net en: J4.2 (Pin_2), R4.2
- new net enGnd: J4.1 (Pin_1), U1.2

Commit message: AbcStop Cleanup And Minor code change
Connections:
- net Left_OUT: now also J2.2 (Pin_2); no longer J2.1 (Pin_1)
- net Right_OUT: now also J2.1 (Pin_1); no longer J2.2 (Pin_2)
Other:
- moved on the sheet: J2
Changed lines of the file:
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@@
     )
   )
-  (symbol (lib_id "Connector_Generic:Conn_01x02") (at 229.87 24.13 0) (mirror y) (unit 1)
+  (symbol (lib_id "Connector_Generic:Conn_01x02") (at 229.87 26.67 180) (unit 1)
     (in_bom yes) (on_board yes) (dnp no)
-    (property "Reference" "J2" (at 227.33 24.1299 0)
+    (property "Reference" "J2" (at 227.33 26.6701 0)
       (effects (font (size 1.27 1.27)) (justify left))
     )
-    (property "Value" "SCREW" (at 227.33 26.6699 0)
+    (property "Value" "SCREW" (at 227.33 24.1301 0)
       (effects (font (size 1.27 1.27)) (justify left))
     )
-    (property "Footprint" "TerminalBlock_Phoenix:TerminalBlock_Phoenix_PT-1,5-2-3.5-H_1x02_P3.50mm_Horizontal" (at 229.87 24.13 0)
+    (property "Footprint" "TerminalBlock_Phoenix:TerminalBlock_Phoenix_PT-1,5-2-3.5-H_1x02_P3.50mm_Horizontal" (at 229.87 26.67 0)
       (effects (font (size 1.27 1.27)) hide)
     )
-    (property "Datasheet" "~" (at 229.87 24.13 0)
+    (property "Datasheet" "~" (at 229.87 26.67 0)
       (effects (font (size 1.27 1.27)) hide)
     )
