File: Interfaces/LocoBufferEsp32/board/LocoBufferEsp32Craddle/LocoNetInterface.kicad_sch (KiCad schematic)
At the start: 18 parts, among them J2 RJ12, J3 RJ12, Q1 SS8050, Q2 SS8050, U1 LM311

Commit message: LocoCradle
Connections:
- net RSyncA: now reaches J2.1, J3.1
- net RSyncB: now reaches J2.6, J3.6
Changed lines of the file:
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@@
   (junction (at 119.38 54.61) (diameter 0) (color 0 0 0 0)
   )
+  (junction (at 58.42 45.72) (diameter 0) (color 0 0 0 0)
+  )
   (junction (at 55.88 35.56) (diameter 0) (color 0 0 0 0)
+  )
+  (junction (at 58.42 33.02) (diameter 0) (color 0 0 0 0)
   )
   (no_connect (at 156.21 44.45))
@@
     (stroke (width 0) (type default))
   )
+  (wire (pts (xy 58.42 26.67) (xy 58.42 33.02))
+    (stroke (width 0) (type default))
+  )
   (wire (pts (xy 176.53 85.09) (xy 176.53 87.63))
     (stroke (width 0) (type default))
@@
     (stroke (width 0) (type default))
   )
-  (wire (pts (xy 52.07 33.02) (xy 64.77 33.02))
+  (wire (pts (xy 58.42 45.72) (xy 64.77 45.72))
+    (stroke (width 0) (type default))
+  )
+  (wire (pts (xy 52.07 33.02) (xy 58.42 33.02))
     (stroke (width 0) (type default))
   )
@@
     (stroke (width 0) (type default))
   )
+  (wire (pts (xy 58.42 26.67) (xy 59.69 26.67))
+    (stroke (width 0) (type default))
+  )
   (wire (pts (xy 123.19 104.14) (xy 133.35 104.14))
     (stroke (width 0) (type default))
   )
+  (wire (pts (xy 58.42 55.88) (xy 58.42 45.72))
+    (stroke (width 0) (type default))
+  )
   (wire (pts (xy 55.88 43.18) (xy 64.77 43.18))
     (stroke (width 0) (type default))
@@
     (stroke (width 0) (type default))
   )
-  (wire (pts (xy 60.96 55.88) (xy 71.12 55.88))
+  (wire (pts (xy 60.96 53.34) (xy 71.12 53.34))
     (stroke (width 0) (type default))
   )
@@
     (stroke (width 0) (type default))
   )
-  (wire (pts (xy 60.96 40.64) (xy 60.96 55.88))
+  (wire (pts (xy 60.96 40.64) (xy 60.96 53.34))
     (stroke (width 0) (type default))
   )
@@
     (stroke (width 0) (type default))
   )
+  (wire (pts (xy 71.12 55.88) (xy 58.42 55.88))
+    (stroke (width 0) (type default))
+  )
   (wire (pts (xy 60.96 40.64) (xy 64.77 40.64))
     (stroke (width 0) (type default))
@@
     (stroke (width 0) (type default))
   )
+  (wire (pts (xy 58.42 33.02) (xy 64.77 33.02))
+    (stroke (width 0) (type default))
+  )
   (wire (pts (xy 55.88 43.18) (xy 55.88 55.88))
     (stroke (width 0) (type default))
@@
     (stroke (width 0) (type default))
   )
-  (wire (pts (xy 52.07 45.72) (xy 64.77 45.72))
+  (wire (pts (xy 52.07 45.72) (xy 58.42 45.72))
     (stroke (width 0) (type default))
   )
@@
     (stroke (width 0) (type default))
   )
-  (label "loconet" (at 71.12 55.88 0) (fields_autoplaced)
+  (label "loconet" (at 71.12 53.34 0) (fields_autoplaced)
     (effects (font (size 1.27 1.27)) (justify left bottom))
   )
@@
     (effects (font (size 1.27 1.27)) (justify left bottom))
   )
+  (hierarchical_label "RSyncA" (shape output) (at 71.12 55.88 0) (fields_autoplaced)
+    (effects (font (size 1.27 1.27)) (justify left))
+  )
+  (hierarchical_label "RSyncB" (shape output) (at 59.69 26.67 0) (fields_autoplaced)
+    (effects (font (size 1.27 1.27)) (justify left))
+  )
   (hierarchical_label "LnTx" (shape input) (at 248.92 39.37 0) (fields_autoplaced)
     (effects (font (size 1.27 1.27)) (justify left))
@@
     (effects (font (size 1.27 1.27)) (justify left))
   )
+  (netclass_flag "" (length 2.54) (shape round) (at 59.69 55.88 180) (fields_autoplaced)
+    (effects (font (size 1.27 1.27)) (justify right bottom))
+    (property "Netclass" "Power" (at 60.2996 58.42 0)
+      (effects (font (size 1.27 1.27) italic) (justify left))
+    )
+  )
+  (netclass_flag "" (length 2.54) (shape round) (at 58.42 26.67 0) (fields_autoplaced)
+    (effects (font (size 1.27 1.27)) (justify left bottom))
+    (property "Netclass" "Power" (at 59.0296 24.13 0)
+      (effects (font (size 1.27 1.27) italic) (justify left))
+    )
+  )
   (symbol (lib_id "Connector:RJ12") (at 41.91 40.64 0) (unit 1)

Commit message: CleanUp
Other:
- company: (none) -> Dcc Diy Tools
- title: (none) -> LocoBuffer Esp32
Changed lines of the file:
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@@
 (kicad_sch (version 20230121) (generator eeschema)
   (paper "A4")
+  (title_block
+    (title "LocoBuffer Esp32")
+    (date "2023-07-17")
+    (rev "0.0.1")
+    (company "Dcc Diy Tools")
+  )
   (junction (at 168.91 52.07) (diameter 0) (color 0 0 0 0)
   )
