File: Interfaces/LocoBufferEsp32/board/LocoBufferEsp32/Esp32Supp.kicad_sch (KiCad schematic)
At the start: 27 parts, among them J1 USB_B_Micro, Q3 SS8050-G, Q4 SS8050-G, SW1 SW_Push, SW2 SW_Push, U2 CP2102N-A01-GQFN28, U3 AMS1117-3.3

Commit message: Cleanup
Changed lines of the file:
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@@
+    (stroke (width 0) (type default))
+  )
+  (polyline (pts (xy 195.58 118.11) (xy 195.58 166.37))
     (stroke (width 0) (type default))
   )

Commit message: Upgrade Libs
Parts:
- C1, C2: LCSC (none) -> C45783
- C3: LCSC (none) -> C1779
- C4: value 0.1uF/50V(10%) -> 0.1uF/50V(10%); LCSC (none) -> C49678
- C5, C6: LCSC (none) -> C49678
- D3: LCSC (none) -> C124187
- D4, D5, D6: LCSC (none) -> C383211
- D7: value Red -> LED; LCSC (none) -> C2296
- J1: value USB_B_Micro -> 10118193-0001LF; footprint Connector_USB:USB_Micro-B_Wuerth_629105150521 -> AMPHENOL_10118193-0001LF; symbol Connector:USB_B_Micro -> LocoNetInterface:10118193-0001LF; LCSC (none) -> C132562; MANUFACTURER (none) -> Amphenol FCI; MAXIMUM_PACKAGE_HEIGHT (none) -> 2.55 mm; PARTREV (none) -> E; STANDARD (none) -> Manufacturer Recommendations
- Q3, Q4: value SS8050-G -> SS8050; symbol Device:Q_NPN_BCE -> Device:Q_NPN_BEC; LCSC (none) -> C2150
- R12, R19: LCSC (none) -> C212449
- R13, R14: LCSC (none) -> C2936632
- R17: LCSC (none) -> C153391
- R18: LCSC (none) -> C245335
- U2: LCSC (none) -> C964632
- U3: LCSC (none) -> C6186
Connections:
- net DTR: now also Q4.2 (E); no longer Q4.3 (E)
- net EN: now also Q3.3 (C); no longer Q3.2 (C)
- net GND: now also J1.S1 (SHIELD), J1.S2 (SHIELD), J1.S3 (SHIELD), J1.S4 (SHIELD), J1.S5 (SHIELD), J1.S6 (SHIELD); no longer J1.6 (Shield)
- net Io0: now also Q4.3 (C); no longer Q4.2 (C)
- net RTS: now also Q3.2 (E); no longer Q3.3 (E)
Other:
- moved on the sheet: D3

Commit message: Version Modular
Parts:
- SW3: renamed from SW1; footprint Button_Switch_SMD:SW_Push_1P1T_XKB_TS-1187A -> Button_Switch_SMD:SW_SPST_CK_RS282G05A3
- SW4: renamed from SW2; footprint Button_Switch_SMD:SW_Push_1P1T_XKB_TS-1187A -> Button_Switch_SMD:SW_SPST_CK_RS282G05A3
- renumbered C1 to C2, C2 to C3, C5 to C4, C4 to C5, C3 to C6, C6 to C7, D4 to D10, D5 to D11, D6 to D12, D3 to D13, D7 to D9, J1 to J4, Q3 to Q6, Q4 to Q7, R12 to R23, R15 to R24, R16 to R25, R13 to R26, R14 to R27, R17 to R28, R18 to R29, R19 to R30, R20 to R31, U2 to U4
