File: MimicPanel/DriverDesk/DriverDeskTft/TftButtons.kicad_sch (KiCad schematic)
At the start: 20 parts, among them SW1 SW_Push, SW10 SW_Push, SW2 SW_Push, SW3 SW_Push, SW4 SW_Push, SW5 SW_Push, SW6 SW_Push, SW7 SW_Push, SW8 SW_Push, SW9 SW_Push

Commit message: TftModule
Parts:
- SW1, SW10, SW2, SW3, SW4, SW5, SW6, SW7, SW8, SW9: footprint Button_Switch_THT:SW_PUSH_6mm -> Button_Switch_THT:SW_PUSH_6mm_H5mm; LCSC (none) -> C2888764; MPN (none) -> 1825910-6

Commit message: rot enc
Parts:
- added R11, R12, R13, R14: R, Resistor_SMD:R_1206_3216Metric, symbol Device:R
- added SW11: RotaryEncoder_Switch, Rotary_Encoder:RotaryEncoder_Alps_EC11E-Switch_Vertical_H20mm, symbol Device:RotaryEncoder_Switch
- added SW12: SW_Push, Button_Switch_THT:SW_PUSH_6mm_H5mm, symbol Switch:SW_Push
- R1, R10, R2, R3, R4, R5, R6, R7, R8, R9: footprint Resistor_SMD:R_0805_2012Metric -> Resistor_SMD:R_1206_3216Metric
Connections:
- net GND: now also SW11.C, SW11.S2, SW12.2
- net VCC: now also R11.1, R12.1, R13.1, R14.1
- new net btn_H: R11.2, SW12.1
- new net btn_RA: R12.2, SW11.A
- new net btn_RB: R13.2, SW11.B
- new net btn_RS: R14.2, SW11.S1
Other:
- moved on the sheet: R1, R10, R2, R3, R4, R5, R6, R7, R8, R9, SW1, SW10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

Commit message: Update btns
Parts:
- SW11: footprint Rotary_Encoder:RotaryEncoder_Alps_EC11E-Switch_Vertical_H20mm -> DigitalTrains:XDCR_PEC11R-4215F-S0024; symbol Device:RotaryEncoder_Switch -> Device:RotaryEncoder_Switch_MP
Connections:
- net GND: now also SW11.MP
Changed lines of the file:
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@@
 	(wire
 		(pts
+			(xy 248.92 147.32) (xy 248.92 148.59)
+		)
+		(stroke
+			(width 0)
+			(type default)
+		)
+	)
+	(wire
+		(pts
 			(xy 270.51 137.16) (xy 265.43 137.16)
 		)
@@
 	(symbol
 		(lib_id "power:GND")
+		(at 248.92 148.59 0)
+		(unit 1)
+		(exclude_from_sim no)
+		(in_bom yes)
+		(on_board yes)
+		(dnp no)
+		(fields_autoplaced yes)
+		(property "Reference" "#PWR036"
+			(at 248.92 154.94 0)
+			(effects
+				(font
+					(size 1.27 1.27)
+				)
+				(hide yes)
+			)
+		)
+		(property "Value" "GND"
+			(at 248.92 153.67 0)
+			(effects
+				(font
+					(size 1.27 1.27)
+				)
+			)
+		)
+		(property "Footprint" ""
+			(at 248.92 148.59 0)
+			(effects
+				(font
+					(size 1.27 1.27)
+				)
+				(hide yes)
+			)
+		)
+		(property "Datasheet" ""
+			(at 248.92 148.59 0)
+			(effects
+				(font
+					(size 1.27 1.27)
+				)
+				(hide yes)
+			)
+		)
+		(property "Description" "Power symbol creates a global label with name \"GND\" , ground"
+			(at 248.92 148.59 0)
+			(effects
+				(font
+					(size 1.27 1.27)
+				)
+				(hide yes)
+			)
+		)
+		(pin "1"
+		)
+		(instances
+			(project "DriverDeskTft"
+				(path "/c825b4d0-cfb0-42ac-8db7-b9a5afa1d288/f055642a-0437-415d-864a-addd8a4ed87f"
+					(reference "#PWR036")
+					(unit 1)
+				)
+			)
+		)
+	)
+	(symbol
+		(lib_id "power:GND")
 		(at 167.64 157.48 0)
 		(unit 1)
@@
 	)
 	(symbol
-		(lib_id "Device:RotaryEncoder_Switch")
+		(lib_id "Device:RotaryEncoder_Switch_MP")
 		(at 248.92 139.7 0)
 		(unit 1)
@@
 			)
 		)
-		(property "Footprint" "Rotary_Encoder:RotaryEncoder_Alps_EC11E-Switch_Vertical_H20mm"
+		(property "Footprint" "DigitalTrains:XDCR_PEC11R-4215F-S0024"
 			(at 245.11 135.636 0)
 			(effects
@@
 		)
 		(property "Datasheet" "~"
-			(at 248.92 133.096 0)
+			(at 248.92 152.4 0)
 			(effects
 				(font
@@
 			)
 		)
-		(property "Description" "Rotary encoder, dual channel, incremental quadrate outputs, with switch"
-			(at 248.92 139.7 0)
+		(property "Description" "Rotary encoder, dual channel, incremental quadrate outputs, with switch and MP Pin"
+			(at 248.92 154.94 0)
 			(effects
 				(font
@@
 		(pin "S2"
 		)
+		(pin "MP"
+		)
 		(instances

Commit message: Doc and DRC
Other:
- company: (none) -> Dcc DIY Tools
- title: (none) -> Driver Desk TFT
Changed lines of the file:
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@@
 	(generator_version "8.0")
 	(paper "A4")
+	(title_block
+		(title "Driver Desk TFT")
+		(date "2024-08-19")
+		(rev "0.0.1")
+		(company "Dcc DIY Tools")
+	)
 	(junction
 		(at 69.85 97.79)

Commit message: Save add File
Parts:
- renumbered R1 to R201, R2 to R202, R3 to R203, R10 to R204, R9 to R205, R8 to R206, R7 to R207, R6 to R208, R5 to R209, R4 to R210, R11 to R211, R14 to R212, R12 to R213, R13 to R214, SW1 to SW201, SW2 to SW202, SW3 to SW203, SW10 to SW204, SW9 to SW205, SW8 to SW206, SW7 to SW207, SW6 to SW208, SW5 to SW209, SW4 to SW210, SW12 to SW211, SW11 to SW212
Connections:
- net btn_1 renamed BTN_1
- net btn_10 renamed BTN_10
- net btn_2 renamed BTN_2
- net btn_3 renamed BTN_3
- net btn_4 renamed BTN_4
- net btn_5 renamed BTN_5
- net btn_6 renamed BTN_6
- net btn_7 renamed BTN_7
- net btn_8 renamed BTN_8
- net btn_9 renamed BTN_9
- net btn_H renamed RENC_H
- net btn_RA renamed RENC_A
- net btn_RB renamed RENC_B
- net btn_RS renamed RENC_S

Commit message: Recuperacion Esquema
Parts:
- R201, R202, R203, R204, R205, R206, R207, R208, R209, R210, R211, R212, R213, R214: value R -> 10K; footprint Resistor_SMD:R_1206_3216Metric -> Resistor_SMD:R_0805_2012Metric; LCSC (none) -> C17414
Changed lines of the file:
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@@
 			)
 		)
-		(property "Value" "R"
+		(property "Value" "10K"
 			(at 71.12 60.9599 0)
 			(effects
@@
 			)
 		)
-		(property "Footprint" "Resistor_SMD:R_1206_3216Metric"
+		(property "Footprint" "Resistor_SMD:R_0805_2012Metric"
 			(at 66.802 59.69 90)
 			(effects
@@
 			)
 		)
-		(property "LCSC" ""
+		(property "LCSC" "C17414"
 			(at 68.58 59.69 0)
 			(effects
@@
 			)
 		)
-		(property "Value" "R"
+		(property "Value" "10K"
 			(at 229.87 148.5899 0)
 			(effects
@@
 			)
 		)
-		(property "Footprint" "Resistor_SMD:R_1206_3216Metric"
+		(property "Footprint" "Resistor_SMD:R_0805_2012Metric"
 			(at 230.632 147.32 90)
 			(effects
@@
 			)
 		)
-		(property "LCSC" ""
+		(property "LCSC" "C17414"
 			(at 232.41 147.32 0)
 			(effects
@@
 			)
 		)
-		(property "Value" "R"
+		(property "Value" "10K"
 			(at 267.97 133.3499 0)
 			(effects
@@
 			)
 		)
-		(property "Footprint" "Resistor_SMD:R_1206_3216Metric"
+		(property "Footprint" "Resistor_SMD:R_0805_2012Metric"
 			(at 267.208 132.08 90)
 			(effects
@@
 			)
 		)
-		(property "LCSC" ""
+		(property "LCSC" "C17414"
 			(at 265.43 132.08 0)
 			(effects
@@
 			)
 		)
-		(property "Value" "R"
+		(property "Value" "10K"
 			(at 113.03 152.3999 0)
 			(effects
@@
 			)
 		)
-		(property "Footprint" "Resistor_SMD:R_1206_3216Metric"
+		(property "Footprint" "Resistor_SMD:R_0805_2012Metric"
 			(at 108.712 151.13 90)
 			(effects
@@
 			)
 		)
-		(property "LCSC" ""
+		(property "LCSC" "C17414"
 			(at 110.49 151.13 0)
 			(effects
@@
 			)
 		)
-		(property "Value" "R"
+		(property "Value" "10K"
 			(at 189.23 124.4599 0)
 			(effects
@@
 			)
 		)
-		(property "Footprint" "Resistor_SMD:R_1206_3216Metric"
+		(property "Footprint" "Resistor_SMD:R_0805_2012Metric"
 			(at 184.912 123.19 90)
 			(effects
@@
 			)
 		)
-		(property "LCSC" ""
+		(property "LCSC" "C17414"
 			(at 186.69 123.19 0)
 			(effects
@@
 			)
 		)
-		(property "Value" "R"
+		(property "Value" "10K"
 			(at 72.39 124.4599 0)
 			(effects
@@
 			)
 		)
-		(property "Footprint" "Resistor_SMD:R_1206_3216Metric"
+		(property "Footprint" "Resistor_SMD:R_0805_2012Metric"
 			(at 68.072 123.19 90)
 			(effects
@@
 			)
 		)
-		(property "LCSC" ""
+		(property "LCSC" "C17414"
 			(at 69.85 123.19 0)
 			(effects
@@
 			)
 		)
-		(property "Value" "R"
+		(property "Value" "10K"
 			(at 153.67 152.3999 0)
 			(effects
@@
 			)
 		)
-		(property "Footprint" "Resistor_SMD:R_1206_3216Metric"
+		(property "Footprint" "Resistor_SMD:R_0805_2012Metric"
 			(at 149.352 151.13 90)
 			(effects
@@
 			)
 		)
-		(property "LCSC" ""
+		(property "LCSC" "C17414"
 			(at 151.13 151.13 0)
 			(effects
@@
 			)
 		)
-		(property "Value" "R"
+		(property "Value" "10K"
 			(at 33.02 146.0499 0)
 			(effects
@@
 			)
 		)
-		(property "Footprint" "Resistor_SMD:R_1206_3216Metric"
+		(property "Footprint" "Resistor_SMD:R_0805_2012Metric"
 			(at 28.702 144.78 90)
 			(effects
@@
 			)
 		)
-		(property "LCSC" ""
+		(property "LCSC" "C17414"
 			(at 30.48 144.78 0)
 			(effects
@@
 			)
 		)
-		(property "Value" "R"
+		(property "Value" "10K"
 			(at 189.23 63.4999 0)
 			(effects
@@
 			)
 		)
-		(property "Footprint" "Resistor_SMD:R_1206_3216Metric"
+		(property "Footprint" "Resistor_SMD:R_0805_2012Metric"
 			(at 184.912 62.23 90)
 			(effects
@@
 			)
 		)
-		(property "LCSC" ""
+		(property "LCSC" "C17414"
 			(at 186.69 62.23 0)
 			(effects
@@
 			)
 		)
-		(property "Value" "R"
+		(property "Value" "10K"
 			(at 189.23 95.2499 0)
 			(effects
@@
 			)
 		)
-		(property "Footprint" "Resistor_SMD:R_1206_3216Metric"
+		(property "Footprint" "Resistor_SMD:R_0805_2012Metric"
 			(at 184.912 93.98 90)
 			(effects
@@
 			)
 		)
-		(property "LCSC" ""
+		(property "LCSC" "C17414"
 			(at 186.69 93.98 0)
 			(effects
@@
 			)
 		)
-		(property "Value" "R"
+		(property "Value" "10K"
 			(at 234.95 133.3499 0)
 			(effects
@@
 			)
 		)
-		(property "Footprint" "Resistor_SMD:R_1206_3216Metric"
+		(property "Footprint" "Resistor_SMD:R_0805_2012Metric"
 			(at 230.632 132.08 90)
 			(effects
@@
 			)
 		)
-		(property "LCSC" ""
+		(property "LCSC" "C17414"
 			(at 232.41 132.08 0)
 			(effects
@@
 			)
 		)
-		(property "Value" "R"
+		(property "Value" "10K"
 			(at 152.4 33.0199 0)
 			(effects
@@
 			)
 		)
-		(property "Footprint" "Resistor_SMD:R_1206_3216Metric"
+		(property "Footprint" "Resistor_SMD:R_0805_2012Metric"
 			(at 148.082 31.75 90)
 			(effects
@@
 			)
 		)
-		(property "LCSC" ""
+		(property "LCSC" "C17414"
 			(at 149.86 31.75 0)
 			(effects
@@
 			)
 		)
-		(property "Value" "R"
+		(property "Value" "10K"
 			(at 113.03 33.0199 0)
 			(effects
@@
 			)
 		)
-		(property "Footprint" "Resistor_SMD:R_1206_3216Metric"
+		(property "Footprint" "Resistor_SMD:R_0805_2012Metric"
 			(at 108.712 31.75 90)
 			(effects
@@
 			)
 		)
-		(property "LCSC" ""
+		(property "LCSC" "C17414"
 			(at 110.49 31.75 0)
 			(effects
@@
 			)
 		)
-		(property "Value" "R"
+		(property "Value" "10K"
 			(at 72.39 93.9799 0)
 			(effects
@@
 			)
 		)
-		(property "Footprint" "Resistor_SMD:R_1206_3216Metric"
+		(property "Footprint" "Resistor_SMD:R_0805_2012Metric"
 			(at 68.072 92.71 90)
 			(effects
@@
 			)
 		)
-		(property "LCSC" ""
+		(property "LCSC" "C17414"
 			(at 69.85 92.71 0)
 			(effects
