File: MimicPanel/DriverDesk/DriverDeskTft/DriverDeskTft.kicad_sch (KiCad schematic)
At the start: 5 parts

Commit message: Update btns
Other:
- sheet Btn ports: added btn_H, btn_RA, btn_RB, btn_RS; removed none
Changed lines of the file:
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@@
+			)
+		)
+		(pin "btn_H" input
+			(at 30.48 20.32 180)
+			(effects
+				(font
+					(size 1.27 1.27)
+				)
+				(justify left)
+			)
+		)
+		(pin "btn_RB" input
+			(at 30.48 29.21 180)
+			(effects
+				(font
+					(size 1.27 1.27)
+				)
+				(justify left)
+			)
+		)
+		(pin "btn_RA" input
+			(at 30.48 26.67 180)
+			(effects
+				(font
+					(size 1.27 1.27)
+				)
+				(justify left)
+			)
+		)
+		(pin "btn_RS" input
+			(at 30.48 33.02 180)
+			(effects
+				(font
+					(size 1.27 1.27)
+				)
+				(justify left)
 			)
 		)

Commit message: headers
Parts:
- added J1: Conn_01x06, Connector_PinHeader_2.54mm:PinHeader_1x08_P2.54mm_Vertical, symbol Connector_Generic:Conn_01x08
- added J2: Conn_01x04, Connector_PinHeader_2.54mm:PinHeader_1x04_P2.54mm_Vertical, symbol Connector_Generic:Conn_01x04
- added J3: Conn_02x05_Odd_Even, Connector_PinHeader_2.54mm:PinHeader_2x05_P2.54mm_Vertical, symbol Connector_Generic:Conn_02x05_Odd_Even
Connections:
- net GND: now also J1.8 (Pin_8)
- net VCC: now also J1.6 (Pin_6)
- net BL: now reaches U1.18 (BL)
- net BL: now also J1.7 (Pin_7)
- net CLK: now reaches U1.20 (CLK)
- net CLK: now also J1.5 (Pin_5)
- net DIN: now reaches U1.21 (DIN)
- net DIN: now also J1.4 (Pin_4)
- net DC: now reaches U1.22 (D/C)
- net DC: now also J1.3 (Pin_3)
- net CS: now reaches U1.23 (CS)
- net CS: now also J1.2 (Pin_2)
- net RST: now reaches U1.24 (RST)
- net RST: now also J1.1 (Pin_1)
- new net Btn1: J3.1 (Pin_1)
- new net Btn10: J3.2 (Pin_2)
- new net Btn2: J3.3 (Pin_3)
- new net Btn3: J3.5 (Pin_5)
- new net Btn4: J3.7 (Pin_7)
- new net Btn5: J3.9 (Pin_9)
- new net Btn6: J3.10 (Pin_10)
- new net Btn7: J3.8 (Pin_8)
- new net Btn8: J3.6 (Pin_6)
- new net Btn9: J3.4 (Pin_4)
- new net BtnH: J2.1 (Pin_1)
- new net RA: J2.2 (Pin_2)
- new net RB: J2.3 (Pin_3)
- new net RS: J2.4 (Pin_4)
- no-connect marks 0 -> 12
Other:
- moved on the sheet: U1

Commit message: Doc and DRC
Connections:
- no-connect marks 12 -> 10
Other:
- company: (none) -> Dcc DIY Tools
- title: (none) -> Driver Desk TFT
Changed lines of the file:
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@@
 	(generator_version "8.0")
 	(paper "A4")
+	(title_block
+		(title "Driver Desk TFT")
+		(date "2024-08-19")
+		(rev "0.0.1")
+		(company "Dcc DIY Tools")
+	)
 	(junction
 		(at 44.45 87.63)
@@
 	)
 	(junction
+		(at 100.33 59.69)
+		(diameter 0)
+		(color 0 0 0 0)
+	)
+	(junction
+		(at 100.33 62.23)
+		(diameter 0)
+		(color 0 0 0 0)
+	)
+	(junction
 		(at 44.45 82.55)
 		(diameter 0)
@@
 	)
 	(no_connect
-		(at 91.44 95.25)
-	)
-	(no_connect
 		(at 91.44 87.63)
 	)
@@
 		(at 91.44 72.39)
 	)
-	(no_connect
-		(at 91.44 97.79)
-	)
-	(wire
-		(pts
-			(xy 91.44 62.23) (xy 101.6 62.23)
+	(wire
+		(pts
+			(xy 91.44 62.23) (xy 100.33 62.23)
 		)
 		(stroke
@@
 	(wire
 		(pts
+			(xy 100.33 62.23) (xy 101.6 62.23)
+		)
+		(stroke
+			(width 0)
+			(type default)
+		)
+	)
+	(wire
+		(pts
 			(xy 35.56 69.85) (xy 54.61 69.85)
 		)
@@
 	(wire
 		(pts
-			(xy 91.44 59.69) (xy 101.6 59.69)
+			(xy 100.33 59.69) (xy 101.6 59.69)
+		)
+		(stroke
+			(width 0)
+			(type default)
+		)
+	)
+	(wire
+		(pts
+			(xy 91.44 59.69) (xy 100.33 59.69)
 		)
 		(stroke
@@
 					(unit 1)
 				)
+			)
+		)
+	)
+	(symbol
+		(lib_id "power:PWR_FLAG")
+		(at 100.33 62.23 180)
+		(unit 1)
+		(exclude_from_sim no)
+		(in_bom yes)
+		(on_board yes)
+		(dnp no)
+		(fields_autoplaced yes)
+		(property "Reference" "#FLG01"
+			(at 100.33 64.135 0)
+			(effects
+				(font
+					(size 1.27 1.27)
+				)
+				(hide yes)
+			)
+		)
+		(property "Value" "PWR_FLAG"
+			(at 100.33 67.31 0)
+			(effects
+				(font
+					(size 1.27 1.27)
+				)
+			)
+		)
+		(property "Footprint" ""
+			(at 100.33 62.23 0)
+			(effects
+				(font
+					(size 1.27 1.27)
+				)
+				(hide yes)
+			)
+		)
+		(property "Datasheet" "~"
+			(at 100.33 62.23 0)
+			(effects
+				(font
+					(size 1.27 1.27)
+				)
+				(hide yes)
+			)
+		)
+		(property "Description" "Special symbol for telling ERC where power comes from"
+			(at 100.33 62.23 0)
+			(effects
+				(font
+					(size 1.27 1.27)
+				)
+				(hide yes)
+			)
+		)
+		(pin "1"
+		)
+		(instances
+			(project ""
+				(path "/c825b4d0-cfb0-42ac-8db7-b9a5afa1d288"
+					(reference "#FLG01")
+					(unit 1)
+				)
+			)
+		)
+	)
+	(symbol
+		(lib_id "power:PWR_FLAG")
+		(at 100.33 59.69 0)
+		(unit 1)
+		(exclude_from_sim no)
+		(in_bom yes)
+		(on_board yes)
+		(dnp no)
+		(fields_autoplaced yes)
+		(property "Reference" "#FLG02"
+			(at 100.33 57.785 0)
+			(effects
+				(font
+					(size 1.27 1.27)
+				)
+				(hide yes)
+			)
+		)
+		(property "Value" "PWR_FLAG"
+			(at 100.33 54.61 0)
+			(effects
+				(font
+					(size 1.27 1.27)
+				)
+			)
+		)
+		(property "Footprint" ""
+			(at 100.33 59.69 0)
+			(effects
+				(font
+					(size 1.27 1.27)
+				)
+				(hide yes)
+			)
+		)
+		(property "Datasheet" "~"
+			(at 100.33 59.69 0)
+			(effects
+				(font
+					(size 1.27 1.27)
+				)
+				(hide yes)
+			)
+		)
+		(property "Description" "Special symbol for telling ERC where power comes from"
+			(at 100.33 59.69 0)
+			(effects
+				(font
+					(size 1.27 1.27)
+				)
+				(hide yes)
+			)
+		)
+		(pin "1"
+		)
+		(instances
+			(project "DriverDeskTft"
+				(path "/c825b4d0-cfb0-42ac-8db7-b9a5afa1d288"
+					(reference "#FLG02")
+					(unit 1)
+				)

Commit message: Save add File
Parts:
- removed J2: Conn_01x04, Connector_PinHeader_2.54mm:PinHeader_1x04_P2.54mm_Vertical, symbol Connector_Generic:Conn_01x04
Connections:
- no-connect marks 10 -> 17
Other:
- added sheet STM32F103 (STM32F103CB.kicad_sch)
- added sheet USB (usb.kicad_sch)
- sheet Btn ports: added BTN_1, BTN_10, BTN_2, BTN_3, BTN_4, BTN_5, BTN_6, BTN_7, BTN_8, BTN_9, RENC_A, RENC_B, RENC_H, RENC_S; removed btn_1, btn_10, btn_2, btn_3, btn_4, btn_5, btn_6, btn_7, btn_8, btn_9, btn_H, btn_RA, btn_RB, btn_RS

Commit message: Recuperacion Esquema
Parts:
- removed J1: Conn_01x06, Connector_PinHeader_2.54mm:PinHeader_1x08_P2.54mm_Vertical, symbol Connector_Generic:Conn_01x08
- removed J3: Conn_02x05_Odd_Even, Connector_PinHeader_2.54mm:PinHeader_2x05_P2.54mm_Vertical, symbol Connector_Generic:Conn_02x05_Odd_Even
- added D101: LED, LED_SMD:LED_0805_2012Metric, symbol Device:LED
- added J101: S5B-PH-SM4-TB, Connector_JST:JST_PH_S5B-PH-SM4-TB_1x05-1MP_P2.00mm_Horizontal, symbol Connector_Generic_MountingPin:Conn_01x05_MountingPin
- added JP101, JP102: SolderJumper_2_Bridged, Jumper:SolderJumper-2_P1.3mm_Bridged_RoundedPad1.0x1.5mm, symbol Jumper:SolderJumper_2_Bridged
- added R101: 1K, Resistor_SMD:R_0805_2012Metric, symbol Device:R
- added R102, R103: 10K, Resistor_SMD:R_0805_2012Metric, symbol Device:R
Connections:
- net GND: now also J101.4 (Pin_4), J101.MP (MountPin)
- net VCC: now also J101.1 (Pin_1), R101.1, R102.1, R103.1
- net BL renamed TFT_BL
- net CLK renamed TFT_CLK
- net CS renamed TFT_CS
- net DC renamed TFT_DC
- net DIN renamed TFT_DIN
- net RST renamed TFT_RST
- new net: JP101.2 (B), R103.2
- new net: D101.2 (A), R101.2
- new net: JP102.2 (B), R102.2
- new net I2C_INT: J101.5 (Pin_5)
- new net I2C_SCL: J101.3 (Pin_3), JP101.1 (A)
- new net I2C_SDA: J101.2 (Pin_2), JP102.1 (A)
- new net LED: D101.1 (K)
- no-connect marks 17 -> 23
Other:
- moved on the sheet: U1

Commit message: Start Of Route
Connections:
- net TFT_CLK: now also U1.9 (SCL); no longer U1.20 (CLK)
- net TFT_DC: now also U1.7 (RS); no longer U1.22 (D/C)
- net TFT_DIN: now also U1.8 (SDA); no longer U1.21 (DIN)
