File: MimicPanel/DriverDesk/DriverDeskTft/STM32F103CB.kicad_sch (KiCad schematic)
At the start: 25 parts, among them J7 Conn_01x06_P1.27, SW2 SW_DIP_x02

Commit message: Start Of Route
Parts:
- removed C? (x2): 1uF, Capacitor_SMD:C_0805_2012Metric, symbol Device:C
- removed C? (x2): 10nF, Capacitor_SMD:C_0805_2012Metric, symbol Device:C
- removed L? (x2): 10uH, Inductor_SMD:L_0805_2012Metric, symbol Device:L
- removed SW2: SW_DIP_x02, Button_Switch_SMD:SW_DIP_SPSTx02_Slide_6.7x6.64mm_W8.61mm_P2.54mm_LowProfile, symbol Switch:SW_DIP_x02
- added JP401, JP402: SolderJumper_2_Open, Jumper:SolderJumper-2_P1.3mm_Open_RoundedPad1.0x1.5mm, symbol Jumper:SolderJumper_2_Open
Connections:
- net GNDA is gone; now on net GND: U?.8 (VSSA)
- net _VDDA is gone; now on net VCC: U?.9 (VDDA)
- net BOOT0: now also JP401.1 (A)
- net PB2: now also JP402.1 (A)
- net VCC: now also JP401.2 (B), JP402.2 (B)
