File: MimicPanel/DriverDesk/DriverDeskTft/usb.kicad_sch (KiCad schematic)
At the start: 6 parts, among them J2 USB_B_Micro

Commit message: Start Of Route
Parts:
- added C301, C302: 10uF, Capacitor_Tantalum_SMD:CP_EIA-3216-18_Kemet-A, symbol Device:C_Polarized
- added U301: AMS1117-3.3, Package_TO_SOT_SMD:SOT-223-3_TabPin2, symbol Regulator_Linear:AMS1117-3.3
Connections:
- net +5V: now also C301.1, U301.3 (VI)
- net GND: now also C301.2, C302.2, U301.1 (GND)
- net VCC: now also C302.1, U301.2 (VO)
